File: protok_ii_rev4.kicad_pcb (KiCad board)
At the start: 2 copper layers, 313.9 x 168.1 mm, 223 parts, among them J1 AudioPlug4, J2 Conn_01x10_Male, J3 Conn_01x04_Male, J4 Conn_01x04_Male, P1 USB_C_Plug, SW1 Rotary_Encoder, U1 proton_c, U2 MCP23017_SO, U3 AT24C256C-SSHL-B

Commit message: convert to kicad 6
Other:
- net class +3V3 removed
- net class Default removed
