File: protok_ii_rev4.kicad_sch (KiCad schematic)
At the start: 207 parts

Commit message: update design
Parts:
- removed BZ1: (no value), symbol Device:Buzzer
- removed J1: (no value), symbol Connector:AudioPlug4
- removed J2: (no value), symbol Connector:Conn_01x10_Male
- removed J3, J4: (no value), symbol Connector:Conn_01x04_Male
- removed P1: (no value), symbol Connector:USB_C_Plug
- removed R3, R6: (no value), symbol Device:R
- removed U1: (no value), symbol proton_c:proton_c
- removed U3: (no value), symbol AT24C256C-SSHL-B:AT24C256C-SSHL-B
- added J7: Conn_01x16_Male, Connector_PinHeader_2.54mm:PinHeader_1x16_P2.54mm_Horizontal, symbol Connector:Conn_01x16_Male
- added J8: Conn_01x12_Female, Connector_PinHeader_2.54mm:PinHeader_1x12_P2.54mm_Horizontal, symbol Connector:Conn_01x12_Female
- added R10, R11, R12, R13, R14, R15, R16, R17, R18, R9: 10K, Resistor_SMD:R_0402_1005Metric, symbol Device:R
- added U3: MCP23017_SO, Package_SO:SOIC-28W_7.5x17.9mm_P1.27mm, symbol Interface_Expansion:MCP23017_SO
- C1, C2: value (none) -> 100nF; footprint (none) -> Capacitor_SMD:C_0402_1005Metric
- D1, D10, D11, D12, D13, D14, D15, D16, D17, D18, D19, D2, D20, D21, D22, D23, D24, D25, D26, D27, D28, D29, D3, D30, D31, D32, D33, D34, D35, D36, D37, D38, D39, D4, D40, D41, D42, D43, D44, D45, D46, D47, D48, D49, D5, D50, D51, D52, D53, D54, D55, D56, D57, D58, D59, D6, D60, D61, D62, D63, D64, D65, D66, D67, D68, D69, D7, D70, D71, D72, D73, D74, D75, D76, D77, D78, D79, D8, D80, D81, D82, D83, D84, D85, D86, D87, D88, D89, D9, D90, D91, D92, D93: value (none) -> 1N4148; footprint (none) -> Diode_SMD:D_SOD-123
- END1, K_ALPHA1, K_ALPHA10, K_ALPHA11, K_ALPHA12, K_ALPHA13, K_ALPHA14, K_ALPHA15, K_ALPHA16, K_ALPHA17, K_ALPHA18, K_ALPHA19, K_ALPHA2, K_ALPHA20, K_ALPHA21, K_ALPHA22, K_ALPHA23, K_ALPHA25, K_ALPHA26, K_ALPHA27, K_ALPHA28, K_ALPHA29, K_ALPHA3, K_ALPHA30, K_ALPHA31, K_ALPHA32, K_ALPHA33, K_ALPHA34, K_ALPHA4, K_ALPHA5, K_ALPHA6, K_ALPHA7, K_ALPHA8, K_ALPHA9, K_DOWN1, K_F1, K_F10, K_F11, K_F12, K_F2, K_F3, K_F4, K_F5, K_F6, K_F7, K_F8, K_F9, K_FN1, K_FN2, K_FN3, K_HOME1, K_INS1, K_LEFT1, K_M1, K_M2, K_M3, K_M4, K_NUM1, K_NUM10, K_NUM11, K_NUM12, K_NUM2, K_NUM3, K_NUM4, K_NUM5, K_NUM6, K_NUM7, K_NUM8, K_NUM9, K_PGDN1, K_PGUP1, K_RIGHT1, K_RSFT1, K_S1, K_S2, K_S3, K_SUPER2, K_TILDE1, K_UP1: value (none) -> MX-NoLED; footprint (none) -> MX_Alps_Choc2_Hybrid:MX-1U
- Joystick1: value (none) -> 2_axis_thumbstick; footprint (none) -> my_lib:2_axis_thumbstick
- K_ALPHA24, K_ALT1, K_ALT2, K_CTRL2, K_ENTER1, K_HYPER1, K_SUPER1: value (none) -> MX-NoLED; footprint (none) -> MX_Alps_Choc2_Hybrid:MX-1.25U
- K_BACKSPACE1, K_DEL1, K_TAB1: value (none) -> MX-NoLED; footprint (none) -> MX_Alps_Choc2_Hybrid:MX-1.5U
- K_CTRL1: value (none) -> MX-NoLED; footprint (none) -> MX_Alps_Choc2_Hybrid:MX-1.75U
- K_LSFT1: value (none) -> MX-NoLED; footprint (none) -> MX_Alps_Choc2_Hybrid:MX-2.25U
- K_SPACE1: value (none) -> MX-NoLED; footprint (none) -> MX_Alps_Choc2_Hybrid:MX-2U
- R1, R2, R4, R5, R7, R8: value (none) -> 10K; footprint (none) -> Resistor_SMD:R_0402_1005Metric
- Rotary1: value (none) -> EC11EBB24C03; footprint (none) -> SamacSys_Parts:EC11EBB24C03
- SW1: value (none) -> Rotary_Encoder; footprint (none) -> my_lib:EC35A1520402
- U2: value (none) -> MCP23017_SO; footprint (none) -> Package_SO:SOIC-28W_7.5x17.9mm_P1.27mm
Connections:
- net +3V3: now also R7.1, R8.1, J8.1 (Pin_1), R10.2, R11.2, R12.2, R13.2, R18.2, R9.2, U3.9 (VDD)
- net Col0: now also J7.1 (Pin_1)
- net Col1: now also J7.2 (Pin_2)
- net Col10: now also J7.11 (Pin_11)
- net Col11: now also J7.12 (Pin_12)
- net Col12: now also J7.13 (Pin_13)
- net Col13: now also J7.14 (Pin_14)
- net Col14: now also J7.15 (Pin_15)
- net Col15: now also J7.16 (Pin_16)
- net Col2: now also J7.3 (Pin_3)
- net Col3: now also J7.4 (Pin_4)
- net Col4: now also J7.5 (Pin_5)
- net Col5: now also J7.6 (Pin_6)
- net Col6: now also J7.7 (Pin_7)
- net Col7: now also J7.8 (Pin_8)
- net Col8: now also J7.9 (Pin_9)
- net Col9: now also J7.10 (Pin_10)
- net GND: now also J8.2 (Pin_2), R14.2, R15.2, R16.2, R17.2, U3.10 (VSS)
- net Row0: now also J8.6 (Pin_6), U3.1 (GPB0)
- net Row1: now also J8.7 (Pin_7), U3.2 (GPB1)
- net Row2: now also J8.8 (Pin_8), U3.3 (GPB2)
- net Row3: now also J8.9 (Pin_9), U3.4 (GPB3)
- net Row4: now also J8.10 (Pin_10), U3.5 (GPB4)
- net Row5: now also J8.11 (Pin_11), U3.6 (GPB5)
- net Row6: now also J8.12 (Pin_12), U3.7 (GPB6)
- net SCL: now also J8.4 (Pin_4), U3.12 (SCK)
- net SDA: now also J8.3 (Pin_3), U3.13 (SDA)
- net at R5.1, U2.15 (A0): no longer U2.16 (A1), U2.17 (A2)
- net at R4.1, U2.18 (~{RESET}): no longer U2.19 (INTB), U2.20 (INTA)
- new net: R16.1, U2.16 (A1)
- new net: R14.1, U2.17 (A2)
- new net: R9.1, U2.19 (INTB)
- new net: R11.1, U2.20 (INTA)
- new net: R10.1, U3.19 (INTB)
- new net: R18.1, U3.15 (A0)
- new net: R17.1, U3.16 (A1)
- new net: R13.1, U3.18 (~{RESET})
- new net: R15.1, U3.17 (A2)
- new net: R12.1, U3.20 (INTA)
- no-connect marks 19 -> 0
Other:
- moved on the sheet: C1, D10, D11, D12, D13, D14, D15, D16, D17, D18, D19, D2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
